Commit message: Update rover workspace packages, launch flows, and DockerHub overview

File: rover_description/urdf/components/zed_macro.urdf.xacro (robot description, xacro)
@@ -1,22 +1,39 @@
 <?xml version="1.0"?>
-<!--
-  Depth camera macro for simulation (standalone, no zed_wrapper dependency)
-  This provides the same frame structure as a ZED camera for compatibility.
--->
 <robot xmlns:xacro="http://wiki.ros.org/xacro">
   <xacro:property name="M_PI" value="3.1415926535897931" />
-  <!-- Material definitions -->
   <material name="depth_camera_mat">
     <color rgba="0.25 0.25 0.25 1.0"/>
   </material>
-  <!--
-    Depth Camera Macro
-    Parameters:
-      - name: the camera's name (e.g., "zed")
-      - baseline: distance between stereo cameras (default 0.12m for ZED2i-like)
-      - height: camera height (default 0.03m)
-  -->
-  <xacro:macro name="depth_camera" params="name=zed baseline=0.12 height=0.03">
-    <!-- Camera mounting point (the threaded screw hole in the bottom) -->
+  <!-- Keep params aligned with zed-ros2-wrapper macro for compatibility. -->
+  <xacro:macro name="zed_camera" params="name=zed model=virtual enable_gnss=false custom_baseline=0.12 gnss_xyz:='0 0 0' gnss_rpy:='0 0 0'">
+    <xacro:if value="${model == 'zed'}">
+      <xacro:property name="baseline" value="0.12" />
+      <xacro:property name="height" value="0.03" />
+      <xacro:property name="bottom_slope" value="0.05" />
+      <xacro:property name="optical_offset_x" value="-0.01" />
+      <xacro:property name="mono" value="false" />
+    </xacro:if>
+    <xacro:if value="${model == 'zed2'}">
+      <xacro:property name="baseline" value="0.12" />
+      <xacro:property name="height" value="0.03" />
+      <xacro:property name="bottom_slope" value="0.05" />
+      <xacro:property name="optical_offset_x" value="-0.01" />
+      <xacro:property name="mono" value="false" />
+    </xacro:if>
+    <xacro:if value="${model == 'virtual'}">
+      <xacro:property name="baseline" value="${custom_baseline}" />
+      <xacro:property name="height" value="0.031" />
+      <xacro:property name="bottom_slope" value="0.0" />
+      <xacro:property name="optical_offset_x" value="0.0" />
+      <xacro:property name="mono" value="false" />
+    </xacro:if>
+    <xacro:if value="${model == 'zedxonegs' or model == 'zedxone4k' or model == 'zedxonehdr'}">
+      <xacro:property name="baseline" value="0.0" />
+      <xacro:property name="height" value="0.031" />
+      <xacro:property name="bottom_slope" value="0.0" />
+      <xacro:property name="optical_offset_x" value="0.0" />
+      <xacro:property name="mono" value="true" />
+    </xacro:if>
+    <!-- Camera mounting point -->
     <link name="${name}_camera_link" />
     <!-- Camera Center -->
@@ -44,34 +61,79 @@
       <parent link="${name}_camera_link"/>
       <child link="${name}_camera_center"/>
-      <origin xyz="0 0 ${height/2}" rpy="0 0 0" />
+      <origin xyz="0 0 ${height/2}" rpy="0 ${bottom_slope} 0" />
     </joint>
-    <!-- Left Camera Frame -->
-    <link name="${name}_left_camera_frame" />
-    <joint name="${name}_left_camera_joint" type="fixed">
-      <parent link="${name}_camera_center"/>
-      <child link="${name}_left_camera_frame"/>
-      <origin xyz="0 ${baseline/2} 0" rpy="0 0 0" />
-    </joint>
-    <!-- Left Camera Optical Frame (Z forward, X right, Y down) -->
-    <link name="${name}_left_camera_frame_optical"/>
-    <joint name="${name}_left_camera_optical_joint" type="fixed">
-      <origin xyz="0 0 0" rpy="-${M_PI/2} 0.0 -${M_PI/2}"/>
-      <parent link="${name}_left_camera_frame"/>
-      <child link="${name}_left_camera_frame_optical"/>
-    </joint>
-    <!-- Right Camera Frame -->
-    <link name="${name}_right_camera_frame" />
-    <joint name="${name}_right_camera_joint" type="fixed">
-      <parent link="${name}_camera_center"/>
-      <child link="${name}_right_camera_frame"/>
-      <origin xyz="0 -${baseline/2} 0" rpy="0 0 0" />
-    </joint>
-    <!-- Right Camera Optical Frame (Z forward, X right, Y down) -->
-    <link name="${name}_right_camera_frame_optical"/>
-    <joint name="${name}_right_camera_optical_joint" type="fixed">
-      <origin xyz="0 0 0" rpy="-${M_PI/2} 0.0 -${M_PI/2}"/>
-      <parent link="${name}_right_camera_frame"/>
-      <child link="${name}_right_camera_frame_optical"/>
-    </joint>
+    <xacro:unless value="${mono}">
+      <!-- Left Camera -->
+      <link name="${name}_left_camera_frame" />
+      <joint name="${name}_left_camera_joint" type="fixed">
+        <parent link="${name}_camera_center"/>
+        <child link="${name}_left_camera_frame"/>
+        <origin xyz="${optical_offset_x} ${baseline/2} 0" rpy="0 0 0" />
+      </joint>
+      <link name="${name}_left_camera_frame_optical"/>
+      <joint name="${name}_left_camera_optical_joint" type="fixed">
+        <origin xyz="0 0 0" rpy="-${M_PI/2} 0.0 -${M_PI/2}"/>
+        <parent link="${name}_left_camera_frame"/>
+        <child link="${name}_left_camera_frame_optical"/>
+      </joint>
+      <link name="${name}_right_camera_frame" />
+      <joint name="${name}_right_camera_joint" type="fixed">
+        <parent link="${name}_camera_center"/>
+        <child link="${name}_right_camera_frame"/>
+        <origin xyz="${optical_offset_x} -${baseline/2} 0" rpy="0 0 0" />
+      </joint>
+      <link name="${name}_right_camera_frame_optical"/>
+      <joint name="${name}_right_camera_optical_joint" type="fixed">
+        <origin xyz="0 0 0" rpy="-${M_PI/2} 0.0 -${M_PI/2}"/>
+        <parent link="${name}_right_camera_frame"/>
+        <child link="${name}_right_camera_frame_optical"/>
+      </joint>
+      <link name="${name}_temp_left_link" />
+      <joint name="${name}_temp_left_joint" type="fixed">
+        <parent link="${name}_left_camera_frame"/>
+        <child link="${name}_temp_left_link"/>
+        <origin xyz="0 0 0" rpy="0 0 0" />
+      </joint>
+      <link name="${name}_temp_right_link" />
+      <joint name="${name}_temp_right_joint" type="fixed">
+        <parent link="${name}_right_camera_frame"/>
+        <child link="${name}_temp_right_link"/>
+        <origin xyz="0 0 0" rpy="0 0 0" />
+      </joint>
+      <link name="${name}_mag_link" />
+      <joint name="${name}_mag_joint" type="fixed">
+        <parent link="${name}_camera_center"/>
+        <child link="${name}_mag_link"/>
+        <origin xyz="0 0 0" rpy="0 0 0" />
+      </joint>
+      <link name="${name}_baro_link" />
+      <joint name="${name}_baro_joint" type="fixed">
+        <parent link="${name}_camera_center"/>
+        <child link="${name}_baro_link"/>
+        <origin xyz="0 0 0" rpy="0 0 0" />
+      </joint>
+    </xacro:unless>
+    <xacro:if value="${mono}">
+      <link name="${name}_camera_frame" />
+      <joint name="${name}_camera_joint" type="fixed">
+        <parent link="${name}_camera_center"/>
+        <child link="${name}_camera_frame"/>
+        <origin xyz="${optical_offset_x} 0 0" rpy="0 0 0" />
+      </joint>
+      <link name="${name}_camera_frame_optical"/>
+      <joint name="${name}_camera_optical_joint" type="fixed">
+        <origin xyz="0 0 0" rpy="-${M_PI/2} 0.0 -${M_PI/2}"/>
+        <parent link="${name}_camera_frame"/>
+        <child link="${name}_camera_frame_optical"/>
+      </joint>
+    </xacro:if>
+    <xacro:if value="${enable_gnss}">
+      <link name="${name}_gnss_link" />
+      <joint name="${name}_gnss_joint" type="fixed">
+        <parent link="${name}_camera_link"/>
+        <child link="${name}_gnss_link"/>
+        <origin xyz="${gnss_xyz}" rpy="${gnss_rpy}" />
+      </joint>
+    </xacro:if>
   </xacro:macro>
 </robot>

File: rover_description/urdf/rover_description.urdf.xacro (robot description, xacro)
@@ -97,9 +97,8 @@
   <xacro:wheel_link name="FR" x_offset="0.35401" y_offset="-1"/>
   <xacro:wheel_link name="FL" x_offset="0.35401" y_offset="1"/>
-  <!-- Depth Camera (simulated stereo camera) -->
-  <xacro:depth_camera
+    <!-- ZED Camera (simulated stereo camera) -->
+    <xacro:zed_camera
       name="$(arg camera_name)"
-      baseline="0.12"
-      height="0.03"/>
+      model="zed2"/>
   <joint name="zed_camera_mount" type="fixed">
     <parent link="base_link"/>
@@ -165,31 +164,21 @@
     <axis xyz="0 0 0" />
   </joint>
-  <!-- GPS Link -->
-<link name="gps_link">
-        <sensor name="navsat" type="navsat">
-          <always_on>true</always_on>
-          <update_rate>1</update_rate>
-          <topic>gps/fix</topic>
-          <gz_frame_id>gps_link</gz_frame_id>
-          <navsat>
-            <position_sensing>
-              <horizontal>
-              <!-- Be carefull setting this.
-              Units in degree not in meters https://github.com/gazebosim/sdformat/issues/1572 -->
-                <noise type="gaussian">
-                  <mean>0.0</mean>
-                  <stddev>0.0</stddev>
-                </noise>
-              </horizontal>
-              <vertical>
-                <noise type="gaussian">
-                  <mean>0.0</mean>
-                  <stddev>0.0</stddev>
-                </noise>
-              </vertical>
-            </position_sensing>
-          </navsat>
-        </sensor>
-      </link>
+  <!-- GPS Link (sensor is defined in rover_gazebo.xacro via <gazebo> extension) -->
+  <link name="gps_link">
+    <inertial>
+      <origin xyz="0 0 0" rpy="0 0 0" />
+      <mass value="0.05" />
+      <inertia ixx="1e-6" ixy="0" ixz="0" iyy="1e-6" iyz="0" izz="1e-6" />
+    </inertial>
+    <visual>
+      <origin xyz="0 0 0" rpy="0 0 0" />
+      <geometry>
+        <box size="0.05 0.05 0.05" />
+      </geometry>
+      <material name="sensor_grey">
+        <color rgba="0.3 0.3 0.3 1.0" />
+      </material>
+    </visual>
+  </link>
 <joint name="gps_joint" type="fixed">
   <origin xyz="0.1 0 0.65" rpy="0 0 0" />  <!-- Positioned above the lidar -->

File: rover_description/urdf/rover_gazebo.xacro (robot description, xacro)
@@ -113,4 +113,31 @@
     </sensor>
   </gazebo>
+  <!-- GPS / NavSat Sensor -->
+  <gazebo reference="gps_link">
+    <sensor name="navsat" type="navsat">
+      <always_on>true</always_on>
+      <update_rate>1</update_rate>
+      <topic>/gps/fix</topic>
+      <gz_frame_id>gps_link</gz_frame_id>
+      <ignition_frame_id>gps_link</ignition_frame_id>
+      <navsat>
+        <position_sensing>
+          <horizontal>
+            <!-- Units are degrees, not meters (sdformat navsat noise is angular) -->
+            <noise type="gaussian">
+              <mean>0.0</mean>
+              <stddev>0.0</stddev>
+            </noise>
+          </horizontal>
+          <vertical>
+            <noise type="gaussian">
+              <mean>0.0</mean>
+              <stddev>0.0</stddev>
+            </noise>
+          </vertical>
+        </position_sensing>
+      </navsat>
+    </sensor>
+  </gazebo>
   <!-- ========================================= -->
   <!-- ZED CAMERA SENSORS FOR GAZEBO SIMULATION -->
@@ -142,5 +169,5 @@
       <gz_frame_id>zed_camera_center</gz_frame_id>
       <ignition_frame_id>zed_camera_center</ignition_frame_id>
-      <topic>zed/zed_node/rgb/image_rect_color</topic>
+      <topic>zed/zed_node/rgb/color/rect/image</topic>
     </sensor>
  </gazebo>
